File: Feather_LORA/Feather_LORA/Feather_LORA.sch (KiCad schematic (older format))
At the start: 7 parts, among them J1 Conn_01x04_Female, J2 Conn_01x02_Male, J3 Conn_01x06_Male, J4 Conn_01x06_Male, J5 Conn_01x06_Male, U1 FGPMMOPA6H_GPS, U2 Feather32u4RFM95

Commit message: Added sma and U.FL connectors for the ant
Parts:
- added AE1: Antenna_Shield, Connector_Coaxial:SMA_Amphenol_132289_EdgeMount, symbol Device:Antenna_Shield
- added AE2: Antenna_Shield, Connector_Coaxial:U.FL_Hirose_U.FL-R-SMT-1_Vertical, symbol Device:Antenna_Shield
Connections:
- net GND: now also AE1.2 (Shield), AE2.2 (Shield)
- net at U1.11 (EX_ANT): now also AE1.1 (A), AE2.1 (A)
Changed lines of the file:
@@
 Wire Wire Line
 	6500 4900 5800 4900
+$Comp
+L Device:Antenna_Shield AE1
+U 1 1 5C291743
+P 6950 2300
+F 0 "AE1" V 6934 2529 50  0000 L CNN
+F 1 "Antenna_Shield" V 7025 2529 50  0000 L CNN
+F 2 "Connector_Coaxial:SMA_Amphenol_132289_EdgeMount" H 6950 2400 50  0001 C CNN
+F 3 "~" H 6950 2400 50  0001 C CNN
+	1    6950 2300
+	0    1    1    0
+$EndComp
+Wire Wire Line
+	5250 2500 6400 2500
+Wire Wire Line
+	6400 2500 6400 2300
+Wire Wire Line
+	6400 2300 6500 2300
+$Comp
+L power:GND #PWR0114
+U 1 1 5C29321B
+P 6750 2400
+F 0 "#PWR0114" H 6750 2150 50  0001 C CNN
+F 1 "GND" H 6755 2227 50  0000 C CNN
+F 2 "" H 6750 2400 50  0001 C CNN
+F 3 "" H 6750 2400 50  0001 C CNN
+	1    6750 2400
+	1    0    0    -1
+$EndComp
+$Comp
+L Device:Antenna_Shield AE2
+U 1 1 5C29327E
+P 7050 1900
+F 0 "AE2" V 7034 2129 50  0000 L CNN
+F 1 "Antenna_Shield" V 7125 2129 50  0000 L CNN
+F 2 "Connector_Coaxial:U.FL_Hirose_U.FL-R-SMT-1_Vertical" H 7050 2000 50  0001 C CNN
+F 3 "~" H 7050 2000 50  0001 C CNN
+	1    7050 1900
+	0    1    1    0
+$EndComp
+Wire Wire Line
+	6500 1900 6850 1900
+$Comp
+L power:GND #PWR0115
+U 1 1 5C293286
+P 6850 2000
+F 0 "#PWR0115" H 6850 1750 50  0001 C CNN
+F 1 "GND" H 6855 1827 50  0000 C CNN
+F 2 "" H 6850 2000 50  0001 C CNN
+F 3 "" H 6850 2000 50  0001 C CNN
+	1    6850 2000
+	1    0    0    -1
+$EndComp
+Wire Wire Line
+	6500 1900 6500 2300
+Connection ~ 6500 2300
+Wire Wire Line
+	6500 2300 6750 2300
 $EndSCHEMATC

Commit message: fixed to do terminal blocks
Parts:
- J3, J4, J5: footprint Connector_PinHeader_2.54mm:PinHeader_1x06_P2.54mm_Vertical -> TerminalBlock_TE-Connectivity:TerminalBlock_TE_282834-6_1x06_P2.54mm_Horizontal
Changed lines of the file:
@@
 F 0 "J3" H 8623 4030 50  0000 R CNN
 F 1 "Conn_01x06_Male" H 8623 4121 50  0000 R CNN
-F 2 "Connector_PinHeader_2.54mm:PinHeader_1x06_P2.54mm_Vertical" H 8650 4150 50  0001 C CNN
+F 2 "TerminalBlock_TE-Connectivity:TerminalBlock_TE_282834-6_1x06_P2.54mm_Horizontal" H 8650 4150 50  0001 C CNN
 F 3 "~" H 8650 4150 50  0001 C CNN
 	1    8650 4150
@@
 F 0 "J4" H 9023 5030 50  0000 R CNN
 F 1 "Conn_01x06_Male" H 9023 5121 50  0000 R CNN
-F 2 "Connector_PinHeader_2.54mm:PinHeader_1x06_P2.54mm_Vertical" H 9050 5150 50  0001 C CNN
+F 2 "TerminalBlock_TE-Connectivity:TerminalBlock_TE_282834-6_1x06_P2.54mm_Horizontal" H 9050 5150 50  0001 C CNN
 F 3 "~" H 9050 5150 50  0001 C CNN
 	1    9050 5150
@@
 F 0 "J5" H 9023 5680 50  0000 R CNN
 F 1 "Conn_01x06_Male" H 9023 5771 50  0000 R CNN
-F 2 "Connector_PinHeader_2.54mm:PinHeader_1x06_P2.54mm_Vertical" H 9050 5800 50  0001 C CNN
+F 2 "TerminalBlock_TE-Connectivity:TerminalBlock_TE_282834-6_1x06_P2.54mm_Horizontal" H 9050 5800 50  0001 C CNN
 F 3 "~" H 9050 5800 50  0001 C CNN
 	1    9050 5800
