File: CyCompute/CyCompute/CyCompute.kicad_pcb (KiCad board)
At the start: 2 copper layers, 100 x 150 mm, 17 parts, among them J1 RJ45, J10 RJ45, J11 RJ45, J12 RJ45, J13 Pi Std header, J2 RJ45, J3 RJ45, J4 RJ45, J5 RJ45, J6 RJ45, J7 RJ45, J8 RJ45, J9 RJ45, U1 LAN9514, U2 P82B715DR, U3 TCA9548APWR

Commit message: rev for review
Parts:
- added C11: CAP100n, Capacitor_SMD:C_0805_2012Metric, F.Cu at (90.5, 126.9)
- added C15: CAP100n, Capacitor_SMD:C_0805_2012Metric, F.Cu at (90.6, 121.8)
- added C8: 15pf, Capacitor_SMD:C_0805_2012Metric, F.Cu at (94.8, 126.7)
- added J14: RJ45, Connector_RJ:RJ45_Amphenol_54602-x08_Horizontal, F.Cu at (104.1, 152.7)
- added J15: RJ11, Connector_RJ:RJ12_Amphenol_54601, F.Cu at (35.2, 47.0)
- added J16: USB_A, Connector_USB:USB_A_CNCTech_1001-011-01101_Horizontal, F.Cu at (66.2, 157.6)
- added J17: USB_A, Connector_USB:USB_A_CNCTech_1001-011-01101_Horizontal, F.Cu at (49.9, 157.6)
- added J18: Conn_01x04_Female, Connector_Molex:Molex_Micro-Fit_3.0_43650-0400_1x04_P3.00mm_Horizontal, F.Cu at (90.8, 158.2)
- added U4: IP4234CZ6, gsg-modules:SOT457, F.Cu at (78.9, 147.4)
- added U5: IP4234CZ6, gsg-modules:SOT457, F.Cu at (49.3, 132.6)
- added U6: PAM2306AYPKE, Package_SO:SOIC-8_3.9x4.9mm_P1.27mm, F.Cu at (60.5, 129.0)
- added U7: SP2526A-2EN-L, Package_SO:SOIC-8_3.9x4.9mm_P1.27mm, F.Cu at (61.7, 137.3)
- J10, J11, J12, J9: value RJ45 -> RJ11; footprint Connector_RJ:RJ45_Amphenol_54602-x08_Horizontal -> Connector_RJ:RJ12_Amphenol_54601
- J13: value Pi Std header -> RJ11; footprint Connector_PinHeader_2.54mm:PinHeader_2x20_P2.54mm_Vertical -> Connector_RJ:RJ12_Amphenol_54601
- J6: value RJ45 -> CAM0; footprint Connector_RJ:RJ45_Amphenol_54602-x08_Horizontal -> cam:FPC_22
- J7: value RJ45 -> CAM1; footprint Connector_RJ:RJ45_Amphenol_54602-x08_Horizontal -> cam:FPC_22
- J8: value RJ45 -> Pi Std header; footprint Connector_RJ:RJ45_Amphenol_54602-x08_Horizontal -> Connector_PinHeader_2.54mm:PinHeader_2x20_P2.54mm_Vertical
- U1: value LAN9514 -> TCA9548APWR; footprint Package_DFN_QFN:QFN-64-1EP_9x9mm_P0.5mm_EP7.3x7.3mm -> Package_SO:TSSOP-24_4.4x7.8mm_P0.65mm
- U2: value P82B715DR -> LAN9514; footprint P82B715DR:P82B715DR -> Package_DFN_QFN:QFN-64-1EP_9x9mm_P0.5mm_EP7.3x7.3mm
- U3: value TCA9548APWR -> P82B715DR; footprint Package_SO:TSSOP-24_4.4x7.8mm_P0.65mm -> P82B715DR:P82B715DR
- moved J10 109.7 mm to (98.2, 47.0), turned to 180 degrees
- moved J8 103.4 mm to (106.7, 66.8)
- moved J5 94.2 mm to (36.8, 129.0), turned to 270 degrees
- moved J6 91.2 mm to (114.7, 61.3), turned to 90 degrees
- moved U3 88.3 mm to (47.6, 54.3)
- moved U1 88.2 mm to (98.3, 59.1), turned to 90 degrees
- moved J7 85.6 mm to (114.8, 129.5), turned to 90 degrees
- moved J3 83.8 mm to (36.8, 109.7), turned to 270 degrees
- moved J9 77.2 mm to (113.7, 46.9)
- moved J1 64.3 mm to (37.5, 56.2), turned to 270 degrees
- moved J4 61.5 mm to (36.8, 91.7), turned to 270 degrees
- moved J2 56.7 mm to (37.2, 73.8)
- moved J13 56.3 mm to (51.3, 47.0), turned to 180 degrees
- moved J11 44.9 mm to (82.6, 47.0), turned to 180 degrees
- moved J12 38.7 mm to (67.1, 47.0), turned to 180 degrees
Connections:
- J1 pad 2: (no net) -> GPIO30
- J1 pad 4: (no net) -> GPIO29
- J1 pad 6: (no net) -> GPIO28
- J1 pad 8: (no net) -> GPIO27
- J10 pad 1: (no net) -> Net-(J10-Pad1)
- J10 pad 2: (no net) -> Net-(J10-Pad2)
- J11 pad 1: (no net) -> Net-(J11-Pad1)
- J11 pad 2: (no net) -> Net-(J11-Pad2)
- J12 pad 1: (no net) -> Net-(J12-Pad1)
- J12 pad 2: (no net) -> Net-(J12-Pad2)
- J13 pad 1: (no net) -> Net-(J13-Pad1)
- J13 pad 2: (no net) -> Net-(J13-Pad2)
- J2 pad 2: (no net) -> GPIO34
- J2 pad 4: (no net) -> GPIO33
- J2 pad 6: (no net) -> GPIO32
- J2 pad 8: (no net) -> GPIO31
- J3 pad 2: (no net) -> GPIO38
- J3 pad 4: (no net) -> GPIO37
- J3 pad 6: (no net) -> GPIO36
- J3 pad 8: (no net) -> GPIO35
- J4 pad 2: (no net) -> GPIO43
- J4 pad 4: (no net) -> GPIO42
- J4 pad 6: (no net) -> GPIO41
- J4 pad 8: (no net) -> GPIO39
- J5 pad 6: (no net) -> GPIO45
- J5 pad 8: (no net) -> GPIO44
- J6 pad 1: (no net) -> GND
- J6 pad 2: (no net) -> CAM0_DN0
- J6 pad 3: (no net) -> CAM0_DP0
- J6 pad 4: (no net) -> GND
- J6 pad 5: (no net) -> CAM0_DN1
- J6 pad 6: (no net) -> CAM0_DP1
- J6 pad 7: (no net) -> GND
- J6 pad 8: (no net) -> CAM0_CN
- J7 pad 1: (no net) -> GND
- J7 pad 2: (no net) -> CAM1_DN0
- J7 pad 3: (no net) -> CAM1_DP0
- J7 pad 4: (no net) -> GND
- J7 pad 5: (no net) -> CAM1_DN1
- J7 pad 6: (no net) -> CAM1_DP1
- J7 pad 7: (no net) -> GND
- J7 pad 8: (no net) -> CAM1_CN
- J8 pad 1: (no net) -> +3V3
- J8 pad 2: (no net) -> +5V
- J8 pad 3: (no net) -> GPIO02
- J8 pad 4: (no net) -> +5V
- J8 pad 5: (no net) -> GPIO03
- J8 pad 6: (no net) -> GND
- J8 pad 7: (no net) -> GPIO04
- J8 pad 8: (no net) -> GPIO14
- J9 pad 1: (no net) -> Net-(J9-Pad1)
- J9 pad 2: (no net) -> Net-(J9-Pad2)
- MD1 pad 11: (no net) -> GPIO03
- MD1 pad 135: (no net) -> CAM1_DP3
- MD1 pad 136: (no net) -> CAM0_DP0
- MD1 pad 137: (no net) -> CAM1_DN3
- MD1 pad 138: (no net) -> CAM0_DN0
- MD1 pad 141: (no net) -> CAM1_DP2
- MD1 pad 142: (no net) -> CAM0_CP
- MD1 pad 143: (no net) -> CAM1_DN2
- MD1 pad 144: (no net) -> CAM0_CN
- MD1 pad 147: (no net) -> CAM1_CP
- MD1 pad 148: (no net) -> CAM0_DP1
- MD1 pad 149: (no net) -> CAM1_CN
- MD1 pad 15: (no net) -> GPIO04
- MD1 pad 150: (no net) -> CAM0_DN1
- MD1 pad 153: (no net) -> CAM1_DP1
- MD1 pad 155: (no net) -> CAM1_DN1
- MD1 pad 159: (no net) -> CAM1_DP0
- MD1 pad 161: (no net) -> CAM1_DN0
- MD1 pad 165: (no net) -> USBDP0
- MD1 pad 167: (no net) -> USBDM0
- MD1 pad 17: (no net) -> GPIO05
- MD1 pad 183: (no net) -> +1V8
- MD1 pad 184: (no net) -> +1V8
- MD1 pad 185: (no net) -> +1V8
- MD1 pad 186: (no net) -> +1V8
- MD1 pad 189: (no net) -> +3V3
- MD1 pad 190: (no net) -> +3V3
- MD1 pad 191: (no net) -> +3V3
- MD1 pad 192: (no net) -> +3V3
- MD1 pad 193: (no net) -> +3V3
- MD1 pad 194: (no net) -> +3V3
- MD1 pad 197: (no net) -> +5V
- MD1 pad 198: (no net) -> +5V
- MD1 pad 199: (no net) -> +5V
- MD1 pad 200: (no net) -> +5V
- MD1 pad 21: (no net) -> GPIO06
- MD1 pad 23: (no net) -> GPIO07
- MD1 pad 27: (no net) -> GPIO08
- MD1 pad 28: (no net) -> GPIO28
- MD1 pad 29: (no net) -> GPIO09
- MD1 pad 30: (no net) -> GPIO29
- MD1 pad 33: (no net) -> GPIO10
- MD1 pad 34: (no net) -> GPIO30
- MD1 pad 35: (no net) -> GPIO11
- MD1 pad 36: (no net) -> GPIO31
- MD1 pad 39: (no net) -> +3V3
- MD1 pad 40: (no net) -> +3V3
- MD1 pad 41: (no net) -> +3V3
- MD1 pad 42: (no net) -> +3V3
- MD1 pad 45: (no net) -> GPIO12
- MD1 pad 46: (no net) -> GPIO32
- MD1 pad 47: (no net) -> GPIO13
- MD1 pad 48: (no net) -> GPIO33
- MD1 pad 51: (no net) -> GPIO14
- MD1 pad 52: (no net) -> GPIO34
- MD1 pad 53: (no net) -> GPIO15
- MD1 pad 54: (no net) -> GPIO35
- MD1 pad 57: (no net) -> GPIO16
- MD1 pad 58: (no net) -> GPIO36
- MD1 pad 59: (no net) -> GPIO17
- MD1 pad 60: (no net) -> GPIO37
- MD1 pad 63: (no net) -> GPIO18
- MD1 pad 64: (no net) -> GPIO38
- MD1 pad 65: (no net) -> GPIO19
- MD1 pad 66: (no net) -> GPIO39
- MD1 pad 69: (no net) -> GPIO20
- MD1 pad 71: (no net) -> GPIO21
- MD1 pad 72: (no net) -> GPIO41
- MD1 pad 75: (no net) -> GPIO22
- MD1 pad 76: (no net) -> GPIO42
- MD1 pad 77: (no net) -> GPIO23
- MD1 pad 78: (no net) -> GPIO43
- MD1 pad 81: (no net) -> GPIO24
- MD1 pad 82: (no net) -> GPIO44
- MD1 pad 83: (no net) -> GPIO25
- MD1 pad 84: (no net) -> GPIO45
- MD1 pad 87: (no net) -> GPIO26
- MD1 pad 89: (no net) -> GPIO27
- MD1 pad 9: (no net) -> GPIO02
- U1 pad 1: (no net) -> GND
- U1 pad 10: Net-(U1-Pad10) -> Net-(J12-Pad2)
- U1 pad 11: (no net) -> Net-(J12-Pad1)
- U1 pad 12: (no net) -> GND
- U1 pad 13: (no net) -> Net-(J13-Pad2)
- U1 pad 14: (no net) -> Net-(J13-Pad1)
- U1 pad 15: Net-(U1-Pad15) -> (no net)
- U1 pad 19: Net-(U1-Pad19) -> SX
- U1 pad 2: (no net) -> GND
- U1 pad 20: (no net) -> SY
- U1 pad 21: (no net) -> GND
- U1 pad 22: (no net) -> GPIO02
- U1 pad 23: (no net) -> GPIO03
- U1 pad 24: (no net) -> +3V3
- U1 pad 4: (no net) -> Net-(J9-Pad2)
- U1 pad 5: Net-(U1-Pad10) -> Net-(J9-Pad1)
- U1 pad 6: (no net) -> Net-(J10-Pad2)
- U1 pad 7: (no net) -> Net-(J10-Pad1)
- U1 pad 8: (no net) -> Net-(J11-Pad2)
- U1 pad 9: (no net) -> Net-(J11-Pad1)
- U2 pad 1: (no net) -> USBDM2
- U2 pad 2: (no net) -> USBDP2
- U2 pad 3: (no net) -> USBDM3
- U2 pad 4: (no net) -> USBDP3
- U2 pad 5: (no net) -> VDD33A
- U3 pad 1: GND -> (no net)
- U3 pad 2: GND -> LX
- U3 pad 3: (no net) -> SX
- U3 pad 4: (no net) -> GND
- U3 pad 6: (no net) -> SY
- U3 pad 7: (no net) -> LY
- U3 pad 8: (no net) -> +3V3
Routing:
- net GND: track 0.00 -> 13.7 mm
- added copper zone on F.Cu, net GND
Other:
- board size 100 x 150 mm -> 100 x 140 mm

Commit message: Getting up to date
Parts:
- moved J16 204.4 mm to (234.3, 41.3), turned to 90 degrees
- moved J17 204.2 mm to (217.8, 41.3), turned to 90 degrees
- moved J5 188.3 mm to (205.1, 44.5), turned to 180 degrees
- moved J3 164.0 mm to (187.3, 44.5), turned to 180 degrees
- moved U2 156.9 mm to (232.4, 66.7)
- moved C8 144.3 mm to (222.5, 59.4)
- moved U5 144.3 mm to (177.0, 65.3)
- moved C11 144.3 mm to (218.1, 59.6)
- moved C15 144.3 mm to (218.2, 54.5)
- moved U4 144.3 mm to (206.6, 80.1)
- moved U7 144.3 mm to (189.4, 70.0)
- moved J18 144.1 mm to (217.8, 90.2)
- moved J14 141.6 mm to (228.6, 85.1)
- moved J4 141.5 mm to (170.2, 44.5), turned to 180 degrees
- moved J2 118.9 mm to (152.4, 44.5), turned to 180 degrees
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Other:
- board size 100 x 140 mm -> 230 x 70 mm
