File: CyCompute/CyCompute/CyCompute.sch (KiCad schematic (older format))
At the start: 3 parts

Commit message: Etho setup
Parts:
- removed U? (x2): MPCIE-Socket, pcie_mini:mpcie-socket, symbol pcie:MPCIE-Socket
- added C? (x12): CAP100n, symbol pspice:CAP
- added C? (x2): CAP 100n, symbol pspice:CAP
- added C?: CAP 4u7/6.3V, symbol pspice:CAP
- added C? (x2): CAP, symbol pspice:CAP
- added C?: CAP0.01uF 50V, symbol pspice:CAP
- added C? (x2): CAP 33p, symbol pspice:CAP
- added D? (x3): LED, symbol Device:LED
- added J1, J10, J11, J12, J2, J3, J4, J5, J6, J7, J8, J9, J?: RJ45, Connector_RJ:RJ45_Amphenol_54602-x08_Horizontal, symbol Connector:RJ45
- added J13: Pi Std header, Connector_PinHeader_2.54mm:PinHeader_2x20_P2.54mm_Vertical, symbol Connector_Generic:Conn_02x20_Odd_Even
- added J?: USB_A, symbol Connector:USB_A
- added L? (x2): INDUCTOR 4.7uH, symbol pspice:INDUCTOR
- added L?: INDUCTOR 4.7 uH, symbol pspice:INDUCTOR
- added R?: R 12K, symbol Device:R
- added R?: R12k4, symbol Device:R
- added R?: 10k, symbol Device:R
- added R?: R10k, symbol Device:R
- added R? (x3): 330, symbol Device:R
- added R?: R 1M, symbol Device:R
- added R?: R 0, symbol Device:R
- added U1: LAN9514, Package_DFN_QFN:QFN-64-1EP_9x9mm_P0.5mm_EP7.3x7.3mm, symbol Interface_Ethernet:LAN9514
- added U2: P82B715DR, P82B715DR:P82B715DR, symbol P82B715DR:P82B715DR
- added U3: TCA9548APWR, Package_SO:TSSOP-24_4.4x7.8mm_P0.65mm, symbol Interface_Expansion:TCA9548APWR
- added U? (x2): IP4234CZ6, gsg-modules:SOT457, symbol ip4234cz6:IP4234CZ6
- added Y?: Crystal 25M, symbol Device:Crystal
- MD1: renamed from MD?; symbol RPi-modules:Board_RPi_CM3lite_200pConnector -> CyCompute-rescue:Board_RPi_CM3lite_200pConnector-RPi-modules
Connections:
- net GND: now reaches MD1.1 (GND)
- net GND: now also MD1.103 (GND), MD1.104 (GND), MD1.109 (GND), MD1.110 (GND), MD1.115 (GND), MD1.116 (GND), MD1.121 (GND), MD1.122 (GND), MD1.127 (GND), MD1.13 (GND), MD1.133 (GND), MD1.134 (GND), MD1.139 (GND), MD1.14 (GND), MD1.140 (GND), MD1.145 (GND), MD1.146 (GND), MD1.151 (GND), MD1.152 (GND), MD1.157 (GND), MD1.163 (GND), MD1.164 (GND), MD1.169 (GND), MD1.170 (GND), MD1.181 (GND), MD1.182 (GND), MD1.187 (GND), MD1.188 (GND), MD1.19 (GND), MD1.195 (GND), MD1.196 (GND), MD1.20 (GND), MD1.25 (GND), MD1.26 (GND), MD1.31 (GND), MD1.32 (GND), MD1.37 (GND), MD1.38 (GND), MD1.43 (GND), MD1.44 (GND), MD1.49 (GND), MD1.50 (GND), MD1.55 (GND), MD1.56 (GND), MD1.61 (GND), MD1.62 (GND), MD1.67 (GND), MD1.68 (GND), MD1.7 (GND), MD1.73 (GND), MD1.74 (GND), MD1.79 (GND), MD1.8 (GND), MD1.80 (GND), MD1.85 (GND), MD1.86 (GND), MD1.91 (GND), MD1.92 (GND), MD1.97 (GND), MD1.98 (GND), C?.2, C?.2, C?.2, C?.2, C?.2, C?.2, C?.2, C?.2, C?.2, C?.2, C?.2, C?.2, C?.2, C?.2, C?.2, C?.2, C?.2, C?.2, C?.2, C?.2, J?.4 (GND), R?.1, R?.2, R?.2, U1.34 (TEST2), U1.44 (CLK24_EN), U1.65 (GND), U3.1 (A0), U3.12 (GND), U3.2 (A1), U3.21 (A2)
- new net: C?.1, R?.2, U1.12 (~RESET)
- new net: R?.2, U1.20 (~FDX_LED~/GPIO0)
- new net: R?.2, U1.21 (~LNKA_LED~/GPIO1)
- new net: R?.2, U1.22 (~SPD_LED~/GPIO2)
- new net: C?.1, R?.2, U1.60 (XO), Y?.1
- new net: C?.1, R?.1, U1.61 (XI), Y?.2
- new net: R?.1, U1.41 (AUTOMDIX_EN)
- new net: R?.1, U1.50 (EXRES)
- new net: R?.1, U1.63 (USBRBIAS)
- new net: D?.1 (K), R?.1 (x3)
- new net +3V3: D?.2 (A), D?.2 (A), D?.2 (A), L?.1, L?.1, R?.1, R?.2, U1.28 (~TRST), U1.29 (TMS), U1.30 (TDI), U1.32 (TCK), U1.40 (TEST3)
- new net GNDS: J?.5 (Shield), R?.2
- new net PRTCTL2: U1.14 (PRTCTL2)
- new net PRTCTL3: U1.16 (PRTCTL3)
- new net PRTCTL4: U1.17 (PRTCTL4)
- new net PRTCTL5: U1.18 (PRTCTL5)
- new net USBDM2: U1.1 (USBDM2)
- new net USBDM3: U1.3 (USBDM3)
- new net USBDM4: U1.6 (USBDM4)
- new net USBDM5: U1.8 (USBDM5)
- new net USBDP2: U1.2 (USBDP2)
- new net USBDP3: U1.4 (USBDP3)
- new net USBDP4: U1.7 (USBDP4)
- new net USBDP5: U1.9 (USBDP5)
- new net VDD18CORE: C?.1, C?.1, C?.1, U1.15 (VDD18CORE), U1.38 (VDD18CORE)
- new net VDD18ETHPLL: C?.1, L?.2, U1.48 (VDD18ETHPLL)
- new net VDD18USBPLL: C?.1, L?.1, U1.62 (VDD18USBPLL)
- new net VDD33A: C?.1, C?.1, C?.1, C?.1, C?.1, C?.1, C?.1, L?.2, U1.10 (VDD33A), U1.49 (VDD33A), U1.5 (VDD33A), U1.51 (VDD33A), U1.54 (VDD33A), U1.57 (VDD33A), U1.64 (VDD33A)
- new net VDD33IO: C?.1, C?.1, C?.1, C?.1, C?.1, L?.2, U1.11 (VBUS_DET), U1.19 (VDD33IO), U1.27 (VDD33IO), U1.33 (VDD33IO), U1.39 (VDD33IO), U1.46 (VDD33IO)
- no-connect marks 0 -> 13

Commit message: rev for review
Parts:
- removed J1, J10, J11, J12, J7, J8, J9: RJ45, Connector_RJ:RJ45_Amphenol_54602-x08_Horizontal, symbol Connector:RJ45
- removed U?: IP4234CZ6, gsg-modules:SOT457, symbol ip4234cz6:IP4234CZ6
- added C10, C7, C8, C9: 15pf, symbol Device:C
- added C14, C17: NF, symbol Device:C
- added C18, C21, C5, C6: 10u, symbol Device:C
- added C23: CAP1u/6.3v, symbol pspice:CAP
- added C29, C34: 100u/10v, symbol pspice:CAP
- added C4: 100n, symbol Device:C
- added J10, J11, J12, J13, J15, J9: RJ11, Connector_RJ:RJ12_Amphenol_54601, symbol Connector:RJ11
- added J17: USB_A, Connector_USB:USB_A_CNCTech_1001-011-01101_Horizontal, symbol Connector:USB_A
- added J18: Conn_01x04_Female, Connector_Molex:Molex_Micro-Fit_3.0_43650-0400_1x04_P3.00mm_Horizontal, symbol Connector:Conn_01x04_Female
- added J6: CAM0, cam:FPC_22, symbol Connector:Conn_01x22_Female
- added J7: CAM1, cam:FPC_22, symbol Connector:Conn_01x22_Female
- added L3, L4: INDUCTOR, symbol pspice:INDUCTOR
- added L6, L7, L8: 4.7uH, symbol pspice:INDUCTOR
- added R1, R2, R3, R4: 1.8k, symbol Device:R
- added R11: 10k, symbol Device:R
- added R15, R16, R17, R18: 49.9, symbol Device:R
- added R22, R5, R6, R7, R8: 100k, symbol Device:R
- added R24, R25: 0, symbol Device:R
- added R26, R27: NF, symbol Device:R
- added U5: IP4234CZ6, gsg-modules:SOT457, symbol ip4234cz6:IP4234CZ6
- added U6: PAM2306AYPKE, SON45P300X300X80-13N, symbol PAM2306AYPKE:PAM2306AYPKE
- added U7: SP2526A-2EN-L, Package_SO:SOIC-8_3.9x4.9mm_P1.27mm, symbol SP2526A-2EN-L:SP2526A-2EN-L
- C11, C15: renamed from C?; footprint (none) -> Capacitor_SMD:C_0805_2012Metric
- J16: renamed from J?; footprint (none) -> Connector_USB:USB_A_CNCTech_1001-011-01101_Horizontal
- gave numbers to parts that had none: 36
- renumbered J6 to J1, J5 to J2, J4 to J3, J3 to J4, J2 to J5, J13 to J8, U3 to U1, U1 to U2, U2 to U3
Connections:
- net +3V3: now also J8.1 (Pin_1), J8.17 (Pin_17), MD1.189 (VDAC), MD1.190 (VDAC), MD1.191 (3V3), MD1.192 (3V3), MD1.193 (3V3), MD1.194 (3V3), MD1.39 (GPIO0-27_VDD), MD1.40 (GPIO0-27_VDD), MD1.41 (GPIO28-45_VDD), MD1.42 (GPIO28-45_VDD), U1.24 (VCC), U3.8 (VCC), C14.1, C18.1, J18.3 (Pin_3), J6.22 (Pin_22), J7.22 (Pin_22), L3.2, R1.1, R11.2, R2.1, R24.1, R3.1, R4.1
- net GND: now also J8.14 (Pin_14), J8.20 (Pin_20), J8.25 (Pin_25), J8.30 (Pin_30), J8.34 (Pin_34), J8.39 (Pin_39), J8.6 (Pin_6), J8.9 (Pin_9), U3.4 (GND), U4.2, C10.1, C18.2, C21.2, C23.1, C29.1, C34.2, C4.2, C5.1, C6.2, C7.1, C8.1, C9.1, J17.4 (GND), J18.4 (Pin_4), J6.1 (Pin_1), J6.10 (Pin_10), J6.13 (Pin_13), J6.16 (Pin_16), J6.19 (Pin_19), J6.4 (Pin_4), J6.7 (Pin_7), J7.1 (Pin_1), J7.10 (Pin_10), J7.13 (Pin_13), J7.16 (Pin_16), J7.19 (Pin_19), J7.4 (Pin_4), J7.7 (Pin_7), L7.2, L8.2, R26.2, R27.2, R5.1, R6.2, R7.1, R8.2, U5.2, U6.13 (EXP), U6.3 (GND@1), U6.9 (GND@2), U7.6 (GND)
- net GNDS: no longer J16.5 (Shield)
- net PRTCTL2: now also U7.1 (ENA), U7.2 (FLGA)
- net PRTCTL3: now also U7.3 (FLGB), U7.4 (ENB)
- net USBDM2: now also U4.6
- net USBDM3: now also U5.6
- net USBDP2: now also U4.1
- net USBDP3: now also U5.1
- net VDD33A: now also R15.2, R16.1, R17.1, R18.2
- net GPIO03: now reaches MD1.11 (GPIO3)
- net GPIO03: now also J8.5 (Pin_5), U1.23 (SDA)
- net CAM1_DP3: now reaches MD1.135 (CAM1_DP3)
- net CAM1_DP3: now also J7.15 (Pin_15)
- net CAM0_DP0: now reaches MD1.136 (CAM0_DP0)
- net CAM0_DP0: now also J6.3 (Pin_3)
- net CAM1_DN3: now reaches MD1.137 (CAM1_DN3)
- net CAM1_DN3: now also J7.14 (Pin_14)
- net CAM0_DN0: now reaches MD1.138 (CAM0_DN0)
- net CAM0_DN0: now also J6.2 (Pin_2)
- net CAM1_DP2: now reaches MD1.141 (CAM1_DP2)
- net CAM1_DP2: now also J7.12 (Pin_12)
- net CAM0_CP: now reaches MD1.142 (CAM0_CP)
- net CAM0_CP: now also J6.9 (Pin_9)
- net CAM1_DN2: now reaches MD1.143 (CAM1_DN2)
- net CAM1_DN2: now also J7.11 (Pin_11)
- net CAM0_CN: now reaches MD1.144 (CAM0_CN)
- net CAM0_CN: now also J6.8 (Pin_8)
- net CAM1_CP: now reaches MD1.147 (CAM1_CP)
- net CAM1_CP: now also J7.9 (Pin_9)
- net CAM0_DP1: now reaches MD1.148 (CAM0_DP1)
- net CAM0_DP1: now also J6.6 (Pin_6)
- net CAM1_CN: now reaches MD1.149 (CAM1_CN)
- net CAM1_CN: now also J7.8 (Pin_8)
- net GPIO04: now reaches MD1.15 (GPIO4)
- net GPIO04: now also J8.7 (Pin_7)
- net CAM0_DN1: now reaches MD1.150 (CAM0_DN1)
- net CAM0_DN1: now also J6.5 (Pin_5)
- net CAM1_DP1: now reaches MD1.153 (CAM1_DP1)
- net CAM1_DP1: now also J7.6 (Pin_6)
- net CAM1_DN1: now reaches MD1.155 (CAM1_DN1)
- net CAM1_DN1: now also J7.5 (Pin_5)
- net CAM1_DP0: now reaches MD1.159 (CAM1_DP0)
- net CAM1_DP0: now also J7.3 (Pin_3)
- net CAM1_DN0: now reaches MD1.161 (CAM1_DN0)
- net CAM1_DN0: now also J7.2 (Pin_2)
- net USBDP0: now reaches MD1.165 (USB_DP)
- net USBDP0: now also U2.59 (USBDP0)
- net USBDM0: now reaches MD1.167 (USB_DM)
- net USBDM0: now also U2.58 (USBDM0)
- net GPIO05: now reaches MD1.17 (GPIO5)
- net GPIO05: now also J8.29 (Pin_29)
- net +1V8: now reaches MD1.183 (1V8)
- net +1V8: now also MD1.184 (1V8), MD1.185 (1V8), MD1.186 (1V8), C17.1, C21.1, L4.2, R25.1
- net +5V: now reaches MD1.197 (VBAT)
- net +5V: now also J8.2 (Pin_2), J8.4 (Pin_4), MD1.198 (VBAT), MD1.199 (VBAT), MD1.200 (VBAT), C5.2, C6.1, J18.2 (Pin_2), L6.1, R22.1, U6.1 (VIN2), U6.6 (EN1), U6.7 (VIN1)
- net GPIO06: now reaches MD1.21 (GPIO6)
- net GPIO06: now also J8.31 (Pin_31)
- net GPIO07: now reaches MD1.23 (GPIO7)
- net GPIO07: now also J8.26 (Pin_26)
- net GPIO08: now reaches MD1.27 (GPIO8)
- net GPIO08: now also J8.24 (Pin_24)
- net GPIO28: now reaches MD1.28 (GPIO28)
- net GPIO28: now also J1.6, R7.2
- net GPIO09: now reaches MD1.29 (GPIO9)
- net GPIO09: now also J8.21 (Pin_21)
- net GPIO00: now reaches MD1.3 (GPIO0)
- net GPIO29: now reaches MD1.30 (GPIO29)
- net GPIO29: now also J1.4, R8.1
- net GPIO10: now reaches MD1.33 (GPIO10)
- net GPIO10: now also J8.19 (Pin_19)
- net GPIO30: now reaches MD1.34 (GPIO30)
- net GPIO30: now also J1.2
- net GPIO11: now reaches MD1.35 (GPIO11)
- net GPIO11: now also J8.23 (Pin_23)
- net GPIO31: now reaches MD1.36 (GPIO31)
- net GPIO31: now also J2.8
- net GPIO12: now reaches MD1.45 (GPIO12)
- net GPIO12: now also J8.32 (Pin_32)
- net GPIO32: now reaches MD1.46 (GPIO32)
- net GPIO32: now also J2.6
- net GPIO13: now reaches MD1.47 (GPIO13)
- net GPIO13: now also J8.33 (Pin_33)
- net GPIO33: now reaches MD1.48 (GPIO33)
- net GPIO33: now also J2.4
- net GPIO01: now reaches MD1.5 (GPIO1)
- net GPIO14: now reaches MD1.51 (GPIO14)
- net GPIO14: now also J8.8 (Pin_8)
- net GPIO34: now reaches MD1.52 (GPIO34)
- net GPIO34: now also J2.2
- net GPIO15: now reaches MD1.53 (GPIO15)
- net GPIO15: now also J8.10 (Pin_10)
- net GPIO35: now reaches MD1.54 (GPIO35)
- net GPIO35: now also J3.8
- net GPIO16: now reaches MD1.57 (GPIO16)
- net GPIO16: now also J8.36 (Pin_36)
- net GPIO36: now reaches MD1.58 (GPIO36)
- net GPIO36: now also J3.6
- net GPIO17: now reaches MD1.59 (GPIO17)
- net GPIO17: now also J8.11 (Pin_11)
- net GPIO37: now reaches MD1.60 (GPIO37)
- net GPIO37: now also J3.4
- net GPIO18: now reaches MD1.63 (GPIO18)
- net GPIO18: now also J8.12 (Pin_12)
- net GPIO38: now reaches MD1.64 (GPIO38)
- net GPIO38: now also J3.2
- net GPIO19: now reaches MD1.65 (GPIO19)
- net GPIO19: now also J8.35 (Pin_35)
- net GPIO39: now reaches MD1.66 (GPIO39)
- net GPIO39: now also J4.8
- net GPIO20: now reaches MD1.69 (GPIO20)
- net GPIO20: now also J8.38 (Pin_38)
- net GPIO40: now reaches MD1.70 (GPIO40)
- net GPIO21: now reaches MD1.71 (GPIO21)
- net GPIO21: now also J8.40 (Pin_40)
- net GPIO41: now reaches MD1.72 (GPIO41)
- net GPIO41: now also J4.6
- net GPIO22: now reaches MD1.75 (GPIO22)
- net GPIO22: now also J8.15 (Pin_15)
- net GPIO42: now reaches MD1.76 (GPIO42)
- net GPIO42: now also J4.4
- net GPIO23: now reaches MD1.77 (GPIO23)
- net GPIO23: now also J8.16 (Pin_16)
- net GPIO43: now reaches MD1.78 (GPIO43)
- net GPIO43: now also J4.2
- net GPIO24: now reaches MD1.81 (GPIO24)
- net GPIO24: now also J8.18 (Pin_18)
- net GPIO44: now reaches MD1.82 (GPIO44)
- net GPIO44: now also J5.8, R5.2
- net GPIO25: now reaches MD1.83 (GPIO25)
- net GPIO25: now also J8.22 (Pin_22)
- net GPIO45: now reaches MD1.84 (GPIO45)
- net GPIO45: now also J5.6, R6.1
- net GPIO26: now reaches MD1.87 (GPIO26)
- net GPIO26: now also J8.37 (Pin_37)
- net GPIO27: now reaches MD1.89 (GPIO27)
- net GPIO27: now also J1.8, J8.13 (Pin_13)
- net GPIO02: now reaches MD1.9 (GPIO2)
- net GPIO02: now also J8.3 (Pin_3), U1.22 (SCL)
- net at U2.52 (RXP): now also J14.3, C8.2, R16.2, R17.2
- net at U2.53 (RXN): now also J14.6, C7.2
- net at U2.55 (TXP): now also J14.1, C10.2
- net at U2.56 (TXN): now also J14.2, C9.2, R15.1, R18.1
- net ID_SD: now reaches J8.27 (Pin_27)
- net ID_SC: now reaches J8.28 (Pin_28)
- net at U1.10 (SD3): now also J12.2
- net at U1.11 (SC3): now also J12.1
- net at U1.13 (SD4): now also J13.2
- net at U1.14 (SC4): now also J13.1
- net SX: now reaches U1.19 (SD7)
- net SX: now also U3.3 (SX)
- net SY: now reaches U1.20 (SC7)
- net SY: now also U3.6 (SY)
- net at U1.3 (~RESET): now also R11.1
- net at U1.4 (SD0): now also J9.2
- net at U1.5 (SC0): now also J9.1
- net at U1.6 (SD1): now also J10.2
- net at U1.7 (SC1): now also J10.1
- net at U1.8 (SD2): now also J11.2
- net at U1.9 (SC2): now also J11.1
- net LX: now reaches U3.2 (LX)
- net LX: now also J15.2
- net LY: now reaches U3.7 (LY)
- net LY: now also J15.1
- net VCC_USB_EX1: now reaches J16.1 (VBUS)
- net VCC_USB_EX1: now also U7.8 (OUTA)
- net USBDM2Out: now reaches J16.2 (D-)
- net USBDM2Out: now also U4.4
- net USBDP2Out: now reaches J16.3 (D+)
- net USBDP2Out: now also U4.3
- net VCC_USB_2: now reaches U4.5
- new net: J16.5 (Shield), L7.1
- new net: C23.2, L6.2, U7.7 (IN)
- new net: J17.5 (Shield), L8.1
- new net: C4.1, R22.2, U6.12 (EN2)
- new net: L4.1, U6.2 (LX2)
- new net: L3.1, U6.8 (LX1)
- new net CAM0_IO0: J6.17 (Pin_17)
- new net CAM0_IO1: J6.18 (Pin_18)
- new net CAM0_SCL: J6.20 (Pin_20), R1.2
- new net CAM0_SDA: J6.21 (Pin_21), R3.2
- new net CAM1_IO0: J7.17 (Pin_17)
- new net CAM1_IO1: J7.18 (Pin_18)
- new net CAM1_SCL: J7.20 (Pin_20), R2.2
- new net CAM1_SDA: J7.21 (Pin_21), R4.2
- new net FB1: C14.2, R24.2, R26.1, U6.4 (FB1)
- new net FB2: C17.2, R25.2, R27.1, U6.10 (FB2)
- new net USBDM3Out: J17.2 (D-), U5.4
- new net USBDP3Out: J17.3 (D+), U5.3
- new net VCC_USB_3: U5.5
- new net VCC_USB_EX2: J17.1 (VBUS), U7.5 (OUTB)
- no-connect marks 13 -> 23
Other:
- note added: "Dont need to populate. Only if emi becomes issue"
- moved on the sheet: C11, C12, C13, C15, C16, C19, C20, C22, C24, C25, C26, C27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

Commit message: Getting up to date
Connections:
- net GND: now also J1.1, J1.3, J1.5, J1.7, J2.1, J2.3, J2.5, J2.7, J3.1, J3.3, J3.5, J3.7, J4.1, J4.3, J4.5, J4.7
Changed lines of the file:
@@
 	1    0    0    -1
 $EndComp
+$Comp
+L power:GND #PWR?
+U 1 1 5D817B58
+P 3400 6650
+F 0 "#PWR?" H 3400 6400 50  0001 C CNN
+F 1 "GND" V 3405 6522 50  0000 R CNN
+F 2 "" H 3400 6650 50  0001 C CNN
+F 3 "" H 3400 6650 50  0001 C CNN
+	1    3400 6650
+	0    -1   -1   0
+$EndComp
+$Comp
+L power:GND #PWR?
+U 1 1 5D817E2E
+P 3400 6850
+F 0 "#PWR?" H 3400 6600 50  0001 C CNN
+F 1 "GND" V 3405 6722 50  0000 R CNN
+F 2 "" H 3400 6850 50  0001 C CNN
+F 3 "" H 3400 6850 50  0001 C CNN
+	1    3400 6850
+	0    -1   -1   0
+$EndComp
+$Comp
+L power:GND #PWR?
+U 1 1 5D82CE72
+P 3400 7050
+F 0 "#PWR?" H 3400 6800 50  0001 C CNN
+F 1 "GND" V 3405 6922 50  0000 R CNN
+F 2 "" H 3400 7050 50  0001 C CNN
+F 3 "" H 3400 7050 50  0001 C CNN
+	1    3400 7050
+	0    -1   -1   0
+$EndComp
+$Comp
+L power:GND #PWR?
+U 1 1 5D841EB6
+P 3400 7250
+F 0 "#PWR?" H 3400 7000 50  0001 C CNN
+F 1 "GND" V 3405 7122 50  0000 R CNN
+F 2 "" H 3400 7250 50  0001 C CNN
+F 3 "" H 3400 7250 50  0001 C CNN
+	1    3400 7250
+	0    -1   -1   0
+$EndComp
+$Comp
+L power:GND #PWR?
+U 1 1 5D856EFA
+P 3400 8050
+F 0 "#PWR?" H 3400 7800 50  0001 C CNN
+F 1 "GND" V 3405 7922 50  0000 R CNN
+F 2 "" H 3400 8050 50  0001 C CNN
+F 3 "" H 3400 8050 50  0001 C CNN
+	1    3400 8050
+	0    -1   -1   0
+$EndComp
+$Comp
+L power:GND #PWR?
+U 1 1 5D86BF3E
+P 3400 8250
+F 0 "#PWR?" H 3400 8000 50  0001 C CNN
+F 1 "GND" V 3405 8122 50  0000 R CNN
+F 2 "" H 3400 8250 50  0001 C CNN
+F 3 "" H 3400 8250 50  0001 C CNN
+	1    3400 8250
+	0    -1   -1   0
+$EndComp
+$Comp
+L power:GND #PWR?
+U 1 1 5D880F82
+P 3400 8450
+F 0 "#PWR?" H 3400 8200 50  0001 C CNN
+F 1 "GND" V 3405 8322 50  0000 R CNN
+F 2 "" H 3400 8450 50  0001 C CNN
+F 3 "" H 3400 8450 50  0001 C CNN
+	1    3400 8450
+	0    -1   -1   0
+$EndComp
+$Comp
+L power:GND #PWR?
+U 1 1 5D895FC6
+P 3400 8650
+F 0 "#PWR?" H 3400 8400 50  0001 C CNN
+F 1 "GND" V 3405 8522 50  0000 R CNN
+F 2 "" H 3400 8650 50  0001 C CNN
+F 3 "" H 3400 8650 50  0001 C CNN
+	1    3400 8650
+	0    -1   -1   0
+$EndComp
+$Comp
+L power:GND #PWR?
+U 1 1 5D8AB5E6
+P 3400 9450
+F 0 "#PWR?" H 3400 9200 50  0001 C CNN
+F 1 "GND" V 3405 9322 50  0000 R CNN
+F 2 "" H 3400 9450 50  0001 C CNN
+F 3 "" H 3400 9450 50  0001 C CNN
+	1    3400 9450
+	0    -1   -1   0
+$EndComp
+$Comp
+L power:GND #PWR?
+U 1 1 5D8C062A
+P 3400 9650
+F 0 "#PWR?" H 3400 9400 50  0001 C CNN
+F 1 "GND" V 3405 9522 50  0000 R CNN
+F 2 "" H 3400 9650 50  0001 C CNN
+F 3 "" H 3400 9650 50  0001 C CNN
+	1    3400 9650
+	0    -1   -1   0
+$EndComp
+$Comp
+L power:GND #PWR?
+U 1 1 5D8D566E
+P 3400 9850
+F 0 "#PWR?" H 3400 9600 50  0001 C CNN
+F 1 "GND" V 3405 9722 50  0000 R CNN
+F 2 "" H 3400 9850 50  0001 C CNN
+F 3 "" H 3400 9850 50  0001 C CNN
+	1    3400 9850
+	0    -1   -1   0
+$EndComp
+$Comp
+L power:GND #PWR?
+U 1 1 5D8EA6B2
+P 3400 10050
+F 0 "#PWR?" H 3400 9800 50  0001 C CNN
+F 1 "GND" V 3405 9922 50  0000 R CNN
+F 2 "" H 3400 10050 50  0001 C CNN
+F 3 "" H 3400 10050 50  0001 C CNN
+	1    3400 10050
+	0    -1   -1   0
+$EndComp
+$Comp
+L power:GND #PWR?
+U 1 1 5D8FFB42
+P 3400 10650
+F 0 "#PWR?" H 3400 10400 50  0001 C CNN
+F 1 "GND" V 3405 10522 50  0000 R CNN
+F 2 "" H 3400 10650 50  0001 C CNN
+F 3 "" H 3400 10650 50  0001 C CNN
+	1    3400 10650
+	0    -1   -1   0
+$EndComp
+$Comp
+L power:GND #PWR?
+U 1 1 5D914B86
+P 3400 10850
+F 0 "#PWR?" H 3400 10600 50  0001 C CNN
+F 1 "GND" V 3405 10722 50  0000 R CNN
+F 2 "" H 3400 10850 50  0001 C CNN
+F 3 "" H 3400 10850 50  0001 C CNN
+	1    3400 10850
+	0    -1   -1   0
+$EndComp
+$Comp
+L power:GND #PWR?
+U 1 1 5D929BCA
+P 3400 11050
+F 0 "#PWR?" H 3400 10800 50  0001 C CNN
+F 1 "GND" V 3405 10922 50  0000 R CNN
+F 2 "" H 3400 11050 50  0001 C CNN
+F 3 "" H 3400 11050 50  0001 C CNN
+	1    3400 11050
+	0    -1   -1   0
+$EndComp
+$Comp
+L power:GND #PWR?
+U 1 1 5D93EC0E
+P 3400 11250
+F 0 "#PWR?" H 3400 11000 50  0001 C CNN
+F 1 "GND" V 3405 11122 50  0000 R CNN
+F 2 "" H 3400 11250 50  0001 C CNN
+F 3 "" H 3400 11250 50  0001 C CNN
+	1    3400 11250
+	0    -1   -1   0
+$EndComp
 $EndSCHEMATC
