File: CyTracker/Feather_LORA/Feather_LORA/Feather_LORA.kicad_pcb (KiCad board)
At the start: 2 copper layers, 100 x 100 mm, 9 parts, among them J1 Conn_01x04_Female, J2 Conn_01x02_Male, J3 Conn_01x06_Male, J4 Conn_01x06_Male, J5 Conn_01x06_Male, U1 FGPMMOPA6H_GPS, U2 Feather32u4RFM95

Commit message: Getting up to date
Parts:
- added J6: Conn_02x20_Top_Bottom, Pin_Headers:Pin_Header_Angled_2x20_Pitch2.54mm, F.Cu at (172.1, 144.8)
