File: CyTracker/Feather_LORA/Feather_LORA/Feather_LORA.sch (KiCad schematic (older format))
At the start: 9 parts, among them J1 Conn_01x04_Female, J2 Conn_01x02_Male, J3 Conn_01x06_Male, J4 Conn_01x06_Male, J5 Conn_01x06_Male, U1 FGPMMOPA6H_GPS, U2 Feather32u4RFM95

Commit message: Getting up to date
Parts:
- added D?: LED, symbol Device:LED
- added J6: Conn_02x20_Top_Bottom, Pin_Headers:Pin_Header_Angled_2x20_Pitch2.54mm, symbol Connector_Generic:Conn_02x20_Odd_Even
- added R?: R330, symbol Device:R
- U1: symbol ultimateGPS_Library:FGPMMOPA6H_GPS -> Feather_LORA-rescue:FGPMMOPA6H_GPS-ultimateGPS_Library
- U2: symbol Feather:Feather32u4RFM95 -> Feather_LORA-rescue:Feather32u4RFM95-Feather
Connections:
- net +3V3: now also J6.1 (Pin_1), J6.17 (Pin_17)
- net +5V: now also J6.2 (Pin_2), J6.4 (Pin_4)
- net GND: now also J6.14 (Pin_14), J6.20 (Pin_20), J6.25 (Pin_25), J6.30 (Pin_30), J6.34 (Pin_34), J6.39 (Pin_39), J6.6 (Pin_6), J6.9 (Pin_9), R?.1
- net at U2.2 (TX): now also U1.10 (RX)
- net at U2.22 (D11): no longer U1.5 (3D-FIX)
- new net: D?.2 (A), U1.5 (3D-FIX)
- new net: D?.1 (K), R?.2
- new net 21: J6.40 (Pin_40)
- new net GPIO02: J6.3 (Pin_3)
- new net GPIO03: J6.5 (Pin_5)
- new net GPIO04: J6.7 (Pin_7)
- new net GPIO05: J6.29 (Pin_29)
- new net GPIO06: J6.31 (Pin_31)
- new net GPIO08: J6.24 (Pin_24), J6.26 (Pin_26)
- new net GPIO09: J6.21 (Pin_21)
- new net GPIO10: J6.19 (Pin_19)
- new net GPIO11: J6.23 (Pin_23)
- new net GPIO12: J6.32 (Pin_32)
- new net GPIO13: J6.33 (Pin_33)
- new net GPIO14: J6.8 (Pin_8)
- new net GPIO15: J6.10 (Pin_10)
- new net GPIO16: J6.36 (Pin_36)
- new net GPIO17: J6.11 (Pin_11)
- new net GPIO18: J6.12 (Pin_12)
- new net GPIO19: J6.35 (Pin_35)
- new net GPIO20: J6.38 (Pin_38)
- new net GPIO22: J6.15 (Pin_15)
- new net GPIO23: J6.16 (Pin_16)
- new net GPIO24: J6.18 (Pin_18)
- new net GPIO25: J6.22 (Pin_22)
- new net GPIO26: J6.37 (Pin_37)
- new net GPIO27: J6.13 (Pin_13)
- new net ID_SC: J6.28 (Pin_28)
- new net ID_SD: J6.27 (Pin_27)
- no-connect marks 0 -> 1
Other:
- note added: "Add backup power option."
- note added: "Blinking status light for fix"
- note added: "Remove these headers. move out to rj45/pi header\nUse jumpers to select opperation ie rj or pi"
- note added: "Reserved for radio"
- note added: "Tx is needed to set mode."
